File: hw/sch_pcb/MPPB01B.kicad_pcb (KiCad board)
At the start: 2 copper layers, 101.1 x 101.1 mm, 27 parts, among them P1 BTH-030-01-F-D-A, P10 SATA7-67491-1030, P11 HEADER_2x05_PARALLEL, P2 BTH-030-01-F-D-A, P3 BTH-030-01-F-D-A, P4 BTH-030-01-F-D-A, P5 SAS_mini_1888174-6, P6 SAS_mini_1888174-6, P7 HEADER_2x13, P9 HEADER_2x03_PARALLEL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

Commit message: Edit PCB
Other:
- rule pad_to_mask_clearance: 0 -> 0.2
Changed lines of the file:
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@@
       (dielectric_constraints no)
     )
-    (pad_to_mask_clearance 0)
-    (solder_mask_min_width 0.25)
+    (pad_to_mask_clearance 0.2)
     (aux_axis_origin 106.68 193.04)
     (pcbplotparams
