File: hw/sch_pcb/MPPB01.kicad_sch (KiCad schematic)
At the start: 12 parts

Commit message: update assets, save as 7
Parts:
- C1, C3, C4: value (none) -> 100nF/16V; footprint (none) -> Capacitor_SMD:C_0805_2012Metric
- C2: value (none) -> 100uF/6V3; footprint (none) -> Capacitor_SMD:C_1210_3225Metric
- D1: value (none) -> M4; footprint (none) -> Diode_SMD:D_SMA
- P10: value (none) -> SATA7-67491-1030; footprint (none) -> Mlab_CON:SATA-7_THT_VERT_2
- P5, P6: value (none) -> SAS_mini_1888174-6; footprint (none) -> Mlab_CON:SAS-mini_TEConnectivity_1888174_Vertical
- P9: value (none) -> HEADER_2x03_PARALLEL; footprint (none) -> Mlab_Pin_Headers:Straight_2x03
- R1, R2: value (none) -> 100; footprint (none) -> Resistor_SMD:R_0805_2012Metric_Pad1.20x1.40mm_HandSolder
- SW1: value (none) -> Prepinac; footprint (none) -> Mlab_SW:SW_PUSH_SMALL
