File: hw/sch_pcb/paracard-power.kicad_sch (KiCad schematic)
At the start: 4 parts

Commit message: update assets, save as 7
Parts:
- P11: value (none) -> HEADER_2x05_PARALLEL; footprint (none) -> Mlab_Pin_Headers:Straight_2x05
- P3: value (none) -> BTH-030-01-F-D-A; footprint (none) -> Mlab_CON:SAMTEC-BTH-030-01-X-D-A
- P7: value (none) -> HEADER_2x13; footprint (none) -> Mlab_Pin_Headers:Straight_2x13
- R3: value (none) -> 10k; footprint (none) -> Resistor_SMD:R_0805_2012Metric_Pad1.20x1.40mm_HandSolder
